File: Kicad/PrettySmallRobot.kicad_pcb (KiCad board)
At the start: 4 copper layers, 26 x 29 mm, 51 parts, among them J1 TYPE-C-31-M-12, J10 Conn_01x02, J8 Conn_01x02, J9 Conn_01x02, U1 DRV8837, U2 DRV8837, U3 MCP73831-2-OT, U4 ESP32-S2, U6 AP2112K-3.3, Y1 12pF/40MHz

Commit message: all nets routed, drc done
Parts:
- C8, C9: moved to F.Cu
- moved C8 11.9 mm to (186.1, 112.9), turned to 0 degrees
- moved C9 10.8 mm to (183.2, 123.3), turned to -90 degrees
- moved C7 5.40 mm to (173.4, 117.6), turned to 0 degrees
- moved C6 5.22 mm to (173.9, 123.2)
- moved C2 4.75 mm to (196.1, 106.2), turned to -90 degrees
- moved C3 4.59 mm to (193.2, 101.7), turned to 180 degrees
- moved R7 0.92 mm to (184.3, 123.3), turned to -90 degrees
- moved U2 0.32 mm to (194.3, 103.9), turned to 90 degrees
- moved D4 0.20 mm to (188.6, 116.7)
- moved R10 0.20 mm to (188.6, 114.6), turned to 90 degrees
- moved L1 0.13 mm to (182.0, 117.6)
Routing:
- net /MOTORB_IN1: track 0.00 -> 57.0 mm, vias 0 -> 1
- net /MOTORB_IN2: track 0.00 -> 56.2 mm, vias 0 -> 1
- net /~{RESET}: track 0.00 -> 25.4 mm, vias 0 -> 2
- net +3V3: track 10.4 -> 26.7 mm, vias 4 -> 12
- net /BOOT: track 0.00 -> 15.4 mm, vias 0 -> 2
- net /MOTORA_IN1: track 0.00 -> 13.1 mm, vias 0 -> 1
- net /MOTORA_IN2: track 0.00 -> 11.6 mm, vias 0 -> 1
- net /VDDA: track 4.21 -> 10.7 mm, vias 1 -> 3
- net /MOTORA_OUT2: track 0.00 -> 5.90 mm
- net /MOTORB_OUT1: track 0.00 -> 5.25 mm
- net /MOTORB_OUT2: track 0.00 -> 5.23 mm
- net /MOTORA_OUT1: track 0.00 -> 5.19 mm
- net +BATT: track 51.0 -> 55.9 mm
- net Net-(J1-PadA5): track 0.00 -> 4.64 mm, vias 0 -> 1
- net Net-(C22-Pad1): track 11.7 -> 15.6 mm
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Other:
- board text added: "+"
- board text added: "BOOT"
- board text added: "RST"

Commit message: update to latest
Parts:
- U3: value MCP73831-2-OT -> MCP73831-2ACI_MC; footprint Package_TO_SOT_SMD:SOT-23-5 -> kicad_footprints:SON50P200X300X100-9N
- moved C12 4.56 mm to (180.5, 102.2), turned to 0 degrees
- moved C21 1.33 mm to (180.5, 106.4), turned to 0 degrees
Connections:
- U3 pad 1: Net-(R5-Pad2) -> /VBUS
- U3 pad 2: GND -> /VBUS
- U3 pad 4: /VBUS -> +BATT
- U3 pad 5: Net-(R6-Pad2) -> Net-(R5-Pad2)
Routing:
- net /VBUS: track 46.4 -> 53.8 mm
- net Net-(R5-Pad2): track 2.51 -> 8.87 mm, vias 0 -> 2
- net Net-(R6-Pad2): track 1.50 -> 2.50 mm, vias 0 -> 2
